File: EagleDesign/full.sch (EAGLE design)
At the start: 19 parts, among them IC1 ATMEGA328-28P, T1 2N3904

Commit message: upload V2 of design
Parts:
- removed IC1: ATMEGA328-28P, atmega328:ATMEGA328-20P
- added ATMEGA328P-AU: ATMEGA328P-AU, Atmel_By_element14_Batch_1-00:ATMEGA328P-AU
- added JP1: (no value), pinhead:PINHD-1X1
- added OPTOCOUPLER: PC817, optocoupler:PC817
- added R3: 220uK, rcl:R-EU_0204/5
- added THERMAL_FUSE: SF70E, discrete:THERMISTOR_R-7,5
- added VARISTOR: 10D391K, varistor:S10K385
- FUSE: value BLX-A -> R3-24; device mylib:BLX-A -> mylib:R3-24
- RELAY: value RELAYPTH -> SRD-05VDC
- renumbered U$1 to RELAY, U$2 to 5V->3.3V
Connections:
- removed net A0: IC1.(PCI8/ADC0)PC0, R2.2
- removed net FUSE_C: FUSE.P$2, U$3.2
- new net D3: ATMEGA328P-AU.PD3, R3.2
- new net FU_IN: FUSE.AC_2, THERMAL_FUSE.2
- new net OPTO_IN: OPTOCOUPLER.A, R3.1
- new net RIN: OPTOCOUPLER.EMIT, R2.2
- new net TR_IN: THERMAL_FUSE.1, U$3.2
- net +5V: now also ATMEGA328P-AU.AVCC, ATMEGA328P-AU.VCC, ATMEGA328P-AU.VCC_2, OPTOCOUPLER.COL; no longer IC1.AVCC, IC1.VCC
- net A1: now also ATMEGA328P-AU.PC1; no longer IC1.(PCI9/ADC1)PC1
- net AC1_F: now also FUSE.AC_1, VARISTOR.1; no longer FUSE.P$1
- net AC2: now also VARISTOR.2
- net AREF: now also ATMEGA328P-AU.AREF; no longer IC1.AREF
- net D10: now also ATMEGA328P-AU.PB2; no longer IC1.(PCI2/SS/OC1B)PB2
- net D2: now also ATMEGA328P-AU.PD2; no longer IC1.(PCI18/INT0)PD2
- net D9: now also ATMEGA328P-AU.PB1; no longer IC1.(PCI1/OC1A/OC1S)PB1
- net GND: now also ATMEGA328P-AU.GND, ATMEGA328P-AU.GND_2, ATMEGA328P-AU.GND_3, OPTOCOUPLER.C; no longer IC1.AGND, IC1.GND
- net MISO: now also ATMEGA328P-AU.PB4; no longer IC1.(PCI4/MISO)PB4
- net MOSI: now also ATMEGA328P-AU.PB3; no longer IC1.(PCI3/MOSI/OC2A)PB3
- net RST: now also ATMEGA328P-AU.PC6, JP1.1; no longer IC1.PC6(/RESET/PCI14)
- net RX: now also ATMEGA328P-AU.PD1; no longer IC1.(PCI17/TXD)PD1
- net SCK: now also ATMEGA328P-AU.PB5; no longer IC1.(PCI5/SCK)PB5
- net TX: now also ATMEGA328P-AU.PD0; no longer IC1.(PCI16/RXD)PD0
